File: kicad-pcb-capteur-deformation/kicad-pcb-capteur-deformation.kicad_sch (KiCad schematic)
At the start: 7 parts, among them J1 Power, J2 Digital/PWM, J3 Analog, J4 Digital/PWM, U3 LTC1050CN8_PBF

Commit message: empreintes et début de wiring KiCad
Parts:
- added C1: 2u, capteur_graphite_lib:C, symbol Device:C
- added C2, C4: 100n, capteur_graphite_lib:C, symbol Device:C
- added M1: Motor_Servo, capteur_graphite_lib:Servo Moteur, symbol Motor:Motor_Servo
- added R1, R3: 100k, capteur_graphite_lib:R, symbol Device:R
- added R2: 1k, capteur_graphite_lib:R, symbol Device:R
- added R4: 10k, capteur_graphite_lib:R, symbol Device:R
- added U4: ~, capteur_graphite_lib:OLED SSD1306, symbol capteur_graphite_lib:OLED_SSD-1306
- added U5: MCP41010-I_P, capteur_graphite_lib:Resistance Variable, symbol capteur_graphite_lib:MCP41010-I_P
- added U6: ~, capteur_graphite_lib:Capteur, symbol capteur_graphite_lib:capteur_graphite
- added U7: ~, capteur_graphite_lib:Flex Sensor, symbol capteur_graphite_lib:Flex_Sensor
- U3: footprint LTC1050CN8_PBF:PDIP-8_N -> capteur_graphite_lib:LTC-1050
Connections:
- net *5 is gone; now on net SW: J4.3 (Pin_3)
- net 2 is gone; now on net CLK: J4.6 (Pin_6)
- net 4 is gone; now on net DT: J4.4 (Pin_4)
- net GND: now also U3.4 (V-), C2.2, C4.2, M1.3 (-), R3.1, U4.1 (GND), U5.4 (VSS), U5.5 (PA0), U5.6 (PW0)
- net VCC: now also U3.7 (V+), M1.2 (+), U4.2 (VCC), U5.8 (VDD), U6.1 (VCC), U7.1 (VCC)
- net PB0: now reaches U3.2 (-IN)
- net PB0: now also C1.1, R1.2, U5.7 (PB0)
- net at U3.3 (+IN): now also C4.1, R3.2, R4.1
- net at U3.6 (OUT): now also C1.2, R1.1, R2.1
- net *10 renamed SS
- net SS: now also U5.1 (~{CS})
- net *11 renamed MOSI
- net MOSI: now also U5.3 (SI)
- net *9 renamed PWM
- net PWM: now also M1.1 (PWM)
- net 13 renamed SCK
- net SCK: now also U5.2 (SCK)
- net A1 renamed FLX
- net FLX: now also U7.2 (OUT)
- net SCL/A5 renamed SCL
- net SCL: now also U4.3 (SCL)
- net SDA/A4 renamed SDA
- net SDA: now also U4.4 (SDA)
- new net: R4.2, U6.2 (Vout)
- new net: C2.1, R2.2
Other:
- moved on the sheet: U1, U2, U3

Commit message: PCB fini
Parts:
- added R5: 47k, capteur_graphite_lib:R, symbol Device:R
- U1: value ~ -> Bluetotth HC05
- U2: value ~ -> Encodeur
- U6: value ~ -> Capteur
- U7: value ~ -> Flex
Connections:
- net A2 is gone; now on net Signal: J3.3 (Pin_3)
- net +5V: now also M1.2 (+), U1.1 (VCC), U2.2 (VCC), U3.7 (V+), U4.2 (VCC), U5.8 (VDD), U6.1 (VCC), U7.1 (VCC)
- net FLX: now also R5.1
- net GND: now also R5.2
- net Signal: now reaches C2.1, R2.2
- removed net VCC: J1.8 (Pin_8), M1.2 (+), U1.1 (VCC), U2.2 (VCC), U3.7 (V+), U4.2 (VCC), U5.8 (VDD), U6.1 (VCC), U7.1 (VCC)
- new net VCC_Arduino: J1.8 (Pin_8)
- no-connect marks 1 -> 15

Commit message: maj des fichiers KiCad, VF préliminaire
Parts:
- C1: value 2u -> 1u; footprint capteur_graphite_lib:C -> capteur_graphite_lib:C - 5,08
Changed lines of the file:
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@@
 			)
 		)
-		(property "Value" "2u"
+		(property "Value" "1u"
 			(at 135.89 123.1899 0)
 			(effects
@@
 			)
 		)
-		(property "Footprint" "capteur_graphite_lib:C"
+		(property "Footprint" "capteur_graphite_lib:C - 5,08"
 			(at 133.0452 125.73 0)
 			(effects
